File: hardware/W27C512Programmer.kicad_sch (KiCad schematic)
At the start: 104 parts, among them J1 CTRL, J2 MSB, J3 LSB, J4 Ext_UART, J5 OLED, J6 VP, J7 SAO, Q1 MMBT3904, Q2 MMBT3906, Q3 MMBT3904, Q4 MMBT3904, Q5 MMBT3904, Q6 MMBT3906, Q7 MMBT3906, Q8 MMBT3906, SW1 RST, SW2 USR, U1 MIC2288, U2 74HC573, U3 74HC573, U4 74HC573, U5 28/32 pin ROM

Commit message: Refactored SCH and bring up to KICAD 8.x
- Schematic changed from A4 to A3
- Reorganized schematic for better readability
- Loaded SCH/PCB so KiCAD uses latest format
Parts:
- removed R20: 22k, Resistor_SMD:R_0603_1608Metric, symbol Device:R_Small
- removed RN8: 4k7, Resistor_SMD:R_Array_Convex_4x0603, symbol Device:R_Pack04
- added R13: 22k, Resistor_SMD:R_0603_1608Metric, symbol Device:R_Small
- added RN6: 4k7, Resistor_SMD:R_Array_Convex_4x0603, symbol Device:R_Pack04
- C11: now not fitted
Connections:
- net A17: no longer D6.2 (A), J1.5 (Pin_5)
- net A18: no longer D7.2 (A), J1.6 (Pin_6)
- net A9_VPP_ENABLE: no longer D3.2 (A), J1.2 (Pin_2)
- net GND: now also R13.2, RN6.1 (R1.1), RN6.2 (R2.1), RN6.3 (R3.1), RN6.4 (R4.1)
- net P1_VPP_ENABLE: no longer D5.2 (A), J1.4 (Pin_4)
- net VPE_ENABLE: no longer D4.2 (A), J1.3 (Pin_3)
- net ~{REG_DISABLE}: no longer D9.2 (A), J1.8 (Pin_8)
- net ~{RW}: no longer D8.2 (A), J1.7 (Pin_7)
- net A15@: now reaches D11.1 (K), JP3.1 (A), U5.3 (A15)
- net A15@: now also R13.1
- net OE@: now reaches D12.1 (K), D29.2 (A), J6.1 (Pin_1), Q6.3 (C), R21.1, U5.24 (OE)
- net A9@: now reaches D10.1 (K), D30.2 (A), J6.2 (Pin_2), Q7.3 (C), R19.1, U5.26 (A9)
- net P1_VPP: now reaches D31.2 (A), J6.3 (Pin_3), JP3.2 (C), Q8.3 (C)
- net at D7.1 (K): now also RN7.6 (R3.2)
- net at Q1.3 (C): now also RN9.8 (R1.2); no longer RN9.1 (R1.1)
- net at RN7.5 (R4.2): now also D6.1 (K); no longer D2.1 (K)
- net at D3.1 (K): now also RN6.6 (R3.2); no longer RN7.6 (R3.2)
- net at D4.1 (K): now also RN6.7 (R2.2); no longer RN7.7 (R2.2)
- net at RN7.8 (R1.2): now also D9.1 (K); no longer D5.1 (K)
- net at Q2.1 (B), R4.2: now also RN9.1 (R1.1); no longer RN9.8 (R1.2)
- net at D8.1 (K): now also RN7.7 (R2.2)
- net A16 renamed VPE_TO_VPP
- net VPE_TO_VPP: no longer D2.2 (A), J1.1 (Pin_1)
- new net: D9.2 (A), J1.8 (Pin_8)
- new net: D6.2 (A), J1.5 (Pin_5)
- new net: D2.2 (A), J1.1 (Pin_1)
- new net: D3.2 (A), J1.2 (Pin_2)
- new net: D4.2 (A), J1.3 (Pin_3)
- new net: D5.2 (A), J1.4 (Pin_4)
- new net: D7.2 (A), J1.6 (Pin_6)
- new net: D8.2 (A), J1.7 (Pin_7)
- new net: D5.1 (K), RN6.8 (R1.2)
- new net: D2.1 (K), RN6.5 (R4.2)
Other:
- moved on the sheet: A1, C1, C10, C2, C3, C4, C5, C6, C7, C8, C9, D1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
